Commit message: Edit launch files: directly launch panda with pedestal

File: franka_env/urdf/panda.urdf.xacro (robot description, xacro)
@@ -84,5 +84,5 @@
         <origin xyz="0 0 0" rpy=" 0 0 0"/>
         <geometry>
-          <box size = "0.2 0.2 1.3"/>
+          <box size = "0.2 0.2 1.0"/>
         </geometry>
       </collision>
@@ -90,5 +90,5 @@
         <origin xyz="0 0 0" rpy=" 0 0 0"/>
         <geometry>
-          <box size = "0.2 0.2 1.3"/>
+          <box size = "0.2 0.2 1.0"/>
         </geometry>
         <material name="red">
@@ -103,10 +103,10 @@
       <parent link="world" />
       <child link = "panda_base" />
-      <origin xyz="0.0 0.0 0.65" rpy="0.0 0.0 0.0" />
+      <origin xyz="0.0 0.0 0.5" rpy="0.0 0.0 0.0" />
     </joint>
     <joint name="panda_joint" type="fixed">
       <parent link="panda_base" />
       <child link = "panda_link0" />
-      <origin xyz="0.0 0.0 0.655" rpy="0.0 0.0 0.0" />
+      <origin xyz="0.0 0.0 0.5" rpy="0.0 0.0 0.0" />
     </joint>
 <!--In-Hand Camera-->

Commit message: Fix: realsense camera

File: franka_env/urdf/panda.urdf.xacro (robot description, xacro)
@@ -110,83 +110,9 @@
       <origin xyz="0.0 0.0 0.5" rpy="0.0 0.0 0.0" />
     </joint>
-<!--In-Hand Camera-->
-    <link name="camera_link">
-        <collision>
-            <origin xyz="0 0 0" rpy="0 0 0"/>
-            <geometry>
-                <!-- <mesh filename="file://$(find project_env)/meshes/D435_Solid.STL"/> -->
-                <box size="0.025 0.1 0.025 "/>
-            </geometry>
-        </collision>
-        <visual>
-            <origin xyz="0 0 0" rpy="0 0 0"/>
-            <geometry>
-                <!-- <mesh filename="file://$(find project_env)/meshes/D435_Solid.STL"/> -->
-                <box size="0.025 0.1 0.025 "/>
-            </geometry>
-        </visual>
-        <inertial>
-            <mass value="1e-5"/>
-            <origin xyz="0 0 0" rpy="0 0 0"/>
-            <inertia ixx="1e-6" ixy="0" ixz="0" iyy="1e-6" iyz="0" izz="1e-6" />
-        </inertial>
-    </link>
-    <joint name="camera_joint" type="fixed">
-      <parent link="end_effector_frame" />
-      <child link = "camera_link" />
-      <origin xyz="-0.075 0.0 0.030" rpy="0.0 0.0 0.0" />
-    </joint>
-    <link name="camera_link_optical" />
-    <joint name="camera_optical_joint" type="fixed">
-        <origin xyz="0 0 0" rpy="-1.57 0 -1.57"/>
-        <parent link="camera_link"/>
-        <child link="camera_link_optical"/>
-    </joint>
-    <gazebo reference="camera_link">
-        <sensor type="depth" name="realsense">
-	        <always_on>1</always_on>
-	        <visualize>true</visualize>
-	        <update_rate>0</update_rate>
-	        <camera>
-	            <horizontal_fov>1.047198</horizontal_fov>
-	            <image>
-	                <width>640</width>
-	                <height>480</height>
-	                <format>B8G8R8</format>  <!--Changed format since channels were inverted, to go back, change to R8G8B8-->
-	            </image>
-	            <clip>
-	                <near>0.01</near>
-	                <far>3</far>
-	            </clip>
-	        </camera>
-	        <plugin name="camera_controller" filename="libgazebo_ros_camera.so">
-	            <baseline>0.2</baseline>
-	            <alwaysOn>true</alwaysOn>
-	            <updateRate>0.0</updateRate>
-	            <cameraName>/realsense</cameraName>
-	            <imageTopicName>/realsense/color/image_raw</imageTopicName>
-	            <cameraInfoTopicName>/realsense/color/camera_info</cameraInfoTopicName>
-	            <depthImageTopicName>/realsense/depth/image_raw</depthImageTopicName>
-	            <depthImageInfoTopicName>/realsense/depth/camera_info</depthImageInfoTopicName>
-	            <pointCloudTopicName>/realsense/depth/points</pointCloudTopicName>
-	            <frameName>camera_link_optical</frameName>
-	            <pointCloudCutoff>0.1</pointCloudCutoff>
-	            <pointCloudCutoffMax>3</pointCloudCutoffMax>
-	            <distortionK1>0</distortionK1>
-	            <distortionK2>0</distortionK2>
-	            <distortionK3>0</distortionK3>
-	            <distortionT1>0</distortionT1>
-	            <distortionT2>0</distortionT2>
-	            <CxPrime>0</CxPrime>
-	            <Cx>0</Cx>
-	            <Cy>0</Cy>
-	            <focalLength>0</focalLength>
-	            <hackBaseline>0</hackBaseline>
-	        </plugin>
-        </sensor>
-    </gazebo>
-    <gazebo reference="camera_link">
-      <material> Gazebo/Red </material>
-    </gazebo>
+  <!-- Realsense D435 -->
+  <xacro:include filename="$(find realsense_ros_gazebo)/xacro/depthcam.xacro"/>
+  <xacro:realsense_d435 sensor_name="d435" parent_link="end_effector_frame" rate="10">
+    <origin rpy="0 0 0 " xyz="-0.075 0.0 0.030"/>
+  </xacro:realsense_d435>
   </xacro:if>
 </robot>

Commit message: Add: gripper attach link

File: franka_env/urdf/panda.urdf.xacro (robot description, xacro)
@@ -110,9 +110,29 @@
       <origin xyz="0.0 0.0 0.5" rpy="0.0 0.0 0.0" />
     </joint>
-  <!-- Realsense D435 -->
-  <xacro:include filename="$(find realsense_ros_gazebo)/xacro/depthcam.xacro"/>
-  <xacro:realsense_d435 sensor_name="d435" parent_link="end_effector_frame" rate="10">
-    <origin rpy="0 0 0 " xyz="-0.075 0.0 0.030"/>
-  </xacro:realsense_d435>
+    <!-- Realsense D435 -->
+    <xacro:include filename="$(find realsense_ros_gazebo)/xacro/depthcam.xacro"/>
+    <xacro:realsense_d435 sensor_name="d435" parent_link="end_effector_frame" rate="10">
+      <origin rpy="0 0 0 " xyz="-0.075 0.0 0.030"/>
+    </xacro:realsense_d435>
+    <!-- Gripper Attacher Link & Joint-->
+    <link name="gripper_attach_link">
+      <inertial>
+          <origin xyz="0 0 0" rpy="0 0 0" />
+          <mass value="0.00001" />
+          <inertia ixx="0.001" ixy="0.0" ixz="0.0" iyy="0.001" iyz="0.0" izz="0.001"/>
+      </inertial>
+      <visual>
+          <geometry>
+          <box size= "0.001 0.001 0.001" />
+          </geometry>
+      </visual>
+    </link>
+    <joint name="gripper_attach_joint" type="prismatic" >
+      <parent link="end_effector_frame" />
+      <child link="gripper_attach_link" />
+      <limit effort="10000" lower="0.0" upper="0.0" velocity="0.0"/>
+      <axis xyz="1 0 0" />
+      <origin xyz="0 0 0" rpy="0 0 0"/>
+    </joint>
   </xacro:if>
 </robot>
