Commit message: removed /controller_manager error
New version of ros2_control cannot handle comments inside of URDFs. Removed comments using <!--.*?-->|#.*?$ regex pattern

File: franka_env/urdf/panda.urdf.xacro (robot description, xacro)
@@ -1,60 +1,10 @@
 <?xml version="1.0"?>
-<!--
-# ===================================== COPYRIGHT ===================================== #
-#                                                                                       #
-#  IFRA (Intelligent Flexible Robotics and Assembly) Group, CRANFIELD UNIVERSITY        #
-#  Created on behalf of the IFRA Group at Cranfield University, United Kingdom          #
-#  E-mail: IFRA@cranfield.ac.uk                                                         #
-#                                                                                       #
-#  Licensed under the Apache-2.0 License.                                               #
-#  You may not use this file except in compliance with the License.                     #
-#  You may obtain a copy of the License at: http://www.apache.org/licenses/LICENSE-2.0  #
-#                                                                                       #
-#  Unless required by applicable law or agreed to in writing, software distributed      #
-#  under the License is distributed on an "as-is" basis, without warranties or          #
-#  conditions of any kind, either express or implied. See the License for the specific  #
-#  language governing permissions and limitations under the License.                    #
-#                                                                                       #
-#  IFRA Group - Cranfield University                                                    #
-#  AUTHORS: Mikel Bueno Viso - Mikel.Bueno-Viso@cranfield.ac.uk                         #
-#           Seemal Asif      - s.asif@cranfield.ac.uk                                   #
-#           Phil Webb        - p.f.webb@cranfield.ac.uk                                 #
-#                                                                                       #
-#  Date: July, 2022.                                                                    #
-#                                                                                       #
-# ===================================== COPYRIGHT ===================================== #
-# ===================================== COPYRIGHT ===================================== #
-#                                                                                       #
-#  Some of the information used to build the ROS2 Panda-Robot .urdf files in this ROS2  #
-#  repository has been taken from the following resources:                              #
-#     - frankaemika/franka_ros2 -> https://github.com/frankaemika/franka_ros2.          #
-#       The original files can be found in the franka_description ROS2 package inside   #
-#       he franka_ros2 GitHub repository.                                               #
-#                                                                                       #
-#  AUTHOR: Franka Emika GmbH - support@franka.de                                        #
-#                                                                                       #
-#  Copyright 2021 Franka Emika GmbH                                                     #
-#  (ORIGINAL LICENSE) -> Licensed under the Apache-2.0 License.                         #
-#                                                                                       #
-#  CHANGES MADE:                                                                        #
-#  Robot information/specifications have been taken, and the code has been modified and #
-#  re-organised in accordance with the ros2_RobotSimulation standards.                  #
-#                                                                                       #
-# ===================================== COPYRIGHT ===================================== #
-# ======= CITE OUR WORK ======= #
-# You can cite our work with the following statement:
-# IFRA (2022) ROS2.0 ROBOT SIMULATION. URL: https://github.com/IFRA-Cranfield/ros2_RobotSimulation.
--->
 <robot xmlns:xacro="http://wiki.ros.org/xacro" name="panda">
-  <!-- ===== ARGUMENTS ===== -->
-  <!-- CELL LAYOUT:  -->
   <xacro:arg name="cell_layout_1" default="false"/>
   <xacro:property name="cell_layout_1" value="$(arg cell_layout_1)"/>
   <xacro:arg name="cell_layout_2" default="false"/>
   <xacro:property name="cell_layout_2" value="$(arg cell_layout_2)"/>
-  <!-- END-EFFECTOR:  -->
   <xacro:arg name="EE_no" default="false"/>
   <xacro:property name="EE_no" value="$(arg EE_no)"/>
-  <!-- Include XACRO-MACRO file of the PANDA ROBOT: -->
   <xacro:include filename="$(find franka_env)/urdf/panda_macro.urdf.xacro"/>
   <xacro:panda
@@ -62,9 +12,5 @@
     EE_no="${EE_no}"
   />
-  <!-- Gazebo world link: -->
   <link name="world"/>
-  <!-- ========== ========== ========== ========== ========== ========== -->
-  <!-- CELL LAYOUT SELECTION: -->
-  <!-- CELL LAYOUT N1) PANDA ROBOT alone: -->
   <xacro:if value="${cell_layout_1}">
     <joint name="world-base_link-fixed" type="fixed">
@@ -73,5 +19,4 @@
     </joint>
   </xacro:if>
-  <!-- CELL LAYOUT N2) PANDA ROBOT on top of a pedestal: -->
   <xacro:if value="${cell_layout_2}">
     <link name='panda_base'>
@@ -110,10 +55,8 @@
       <origin xyz="0.0 0.0 0.5" rpy="0.0 0.0 0.0" />
     </joint>
-    <!-- Realsense D435 -->
-    <xacro:include filename="$(find realsense_ros_gazebo)/xacro/depthcam.xacro"/>
+    <xacro:include filename="/home/soham/llm-grasping-panda/src/realsense_ros_gazebo/xacro/depthcam.xacro"/>
     <xacro:realsense_d435 sensor_name="d435" parent_link="end_effector_frame" rate="10">
       <origin rpy="0 0 0 " xyz="-0.075 0.0 0.030"/>
     </xacro:realsense_d435>
-    <!-- Gripper Attacher Link & Joint-->
     <link name="gripper_attach_link">
       <inertial>

File: franka_env/urdf/panda_macro.urdf.xacro (robot description, xacro)
@@ -1,58 +1,9 @@
 <?xml version="1.0"?>
-<!--
-# ===================================== COPYRIGHT ===================================== #
-#                                                                                       #
-#  IFRA (Intelligent Flexible Robotics and Assembly) Group, CRANFIELD UNIVERSITY        #
-#  Created on behalf of the IFRA Group at Cranfield University, United Kingdom          #
-#  E-mail: IFRA@cranfield.ac.uk                                                         #
-#                                                                                       #
-#  Licensed under the Apache-2.0 License.                                               #
-#  You may not use this file except in compliance with the License.                     #
-#  You may obtain a copy of the License at: http://www.apache.org/licenses/LICENSE-2.0  #
-#                                                                                       #
-#  Unless required by applicable law or agreed to in writing, software distributed      #
-#  under the License is distributed on an "as-is" basis, without warranties or          #
-#  conditions of any kind, either express or implied. See the License for the specific  #
-#  language governing permissions and limitations under the License.                    #
-#                                                                                       #
-#  IFRA Group - Cranfield University                                                    #
-#  AUTHORS: Mikel Bueno Viso - Mikel.Bueno-Viso@cranfield.ac.uk                         #
-#           Seemal Asif      - s.asif@cranfield.ac.uk                                   #
-#           Phil Webb        - p.f.webb@cranfield.ac.uk                                 #
-#                                                                                       #
-#  Date: July, 2022.                                                                    #
-#                                                                                       #
-# ===================================== COPYRIGHT ===================================== #
-# ===================================== COPYRIGHT ===================================== #
-#                                                                                       #
-#  Some of the information used to build the ROS2 Panda-Robot .urdf files in this ROS2  #
-#  repository has been taken from the following resources:                              #
-#     - frankaemika/franka_ros2 -> https://github.com/frankaemika/franka_ros2.          #
-#       The original files can be found in the franka_description ROS2 package inside   #
-#       he franka_ros2 GitHub repository.                                               #
-#                                                                                       #
-#  AUTHOR: Franka Emika GmbH - support@franka.de                                        #
-#                                                                                       #
-#  Copyright 2021 Franka Emika GmbH                                                     #
-#  (ORIGINAL LICENSE) -> Licensed under the Apache-2.0 License.                         #
-#                                                                                       #
-#  CHANGES MADE:                                                                        #
-#  Robot information/specifications have been taken, and the code has been modified and #
-#  re-organised in accordance with the ros2_RobotSimulation standards.                  #
-#                                                                                       #
-# ===================================== COPYRIGHT ===================================== #
-# ======= CITE OUR WORK ======= #
-# You can cite our work with the following statement:
-# IFRA (2022) ROS2.0 ROBOT SIMULATION. URL: https://github.com/IFRA-Cranfield/ros2_RobotSimulation.
--->
 <robot xmlns:xacro="http://wiki.ros.org/xacro">
-  <!-- XACRO-MACRO of PANDA ROBOT: -->
   <xacro:macro name="panda" params="prefix EE_no">
-    <!-- Load PANDA ROBOT TRANSMISSION file: -->
     <xacro:include filename="$(find franka_env)/urdf/panda_transmission.xacro" />
     <xacro:panda_transmission
       prefix=""
     />
-    <!-- Load PANDA ROBOT ROS2_CONTROL file: -->
     <xacro:include filename="$(find franka_env)/urdf/panda_ros2control.xacro" />
     <xacro:panda_ros2control
@@ -60,6 +11,4 @@
       EE_no="${EE_no}"
     />
-    <!-- ***** PANDA ROBOT .urdf SERIAL CHAIN ***** -->
-    <!-- panda_link0 -->
     <link name="panda_link0">
       <inertial>
@@ -84,5 +33,4 @@
       </collision>
     </link>
-    <!-- panda_link1 -->
     <link name="panda_link1">
       <inertial>
@@ -107,5 +55,4 @@
       </collision>
     </link>
-    <!-- panda_joint1 -->
     <joint name="panda_joint1" type="revolute">
       <origin rpy="0 0 0" xyz="0 0 0.333"/>
@@ -116,5 +63,4 @@
       <dynamics damping="50.0" friction="1.0"/>
     </joint>
-    <!-- panda_link2 -->
     <link name="panda_link2">
       <inertial>
@@ -139,5 +85,4 @@
       </collision>
     </link>
-    <!-- panda_joint2 -->
     <joint name="panda_joint2" type="revolute">
       <origin rpy="-1.57079632679 0 0" xyz="0 0 0"/>
@@ -148,5 +93,4 @@
       <dynamics damping="50.0" friction="1.0"/>
     </joint>
-    <!-- panda_link3 -->
     <link name="panda_link3">
       <inertial>
@@ -171,5 +115,4 @@
       </collision>
     </link>
-    <!-- panda_joint3 -->
     <joint name="panda_joint3" type="revolute">
       <origin rpy="1.57079632679 0 0" xyz="0 -0.316 0"/>
@@ -180,5 +123,4 @@
       <dynamics damping="10.0" friction="1.0"/>
     </joint>
-    <!-- panda_link4-->
     <link name="panda_link4">
       <inertial>
@@ -203,5 +145,4 @@
       </collision>
     </link>
-    <!-- panda_joint4 -->
     <joint name="panda_joint4" type="revolute">
       <origin rpy="1.57079632679 0 0" xyz="0.0825 0 0"/>
@@ -210,8 +151,6 @@
       <axis xyz="0 0 1"/>
       <limit effort="87" lower="-3.0718" upper="0.0698" velocity="2.1750"/>
-      <!-- upper should be -0.0698, but that brakes simulation when initial position for this joint is 0.0 -->
       <dynamics damping="10.0" friction="1.0"/>
     </joint>
-    <!-- panda_link5 -->
     <link name="panda_link5">
       <inertial>
@@ -236,5 +175,4 @@
       </collision>
     </link>
-    <!-- panda_joint5 -->
     <joint name="panda_joint5" type="revolute">
       <origin rpy="-1.57079632679 0 0" xyz="-0.0825 0.384 0"/>
@@ -245,5 +183,4 @@
       <dynamics damping="5.0" friction="1.0"/>
     </joint>
-    <!-- panda_link6 -->
     <link name="panda_link6">
       <inertial>
@@ -268,7 +205,6 @@
       </collision>
     </link>
-    <!-- panda_joint6 -->
     <joint name="panda_joint6" type="revolute">
-      <origin rpy="1.57079632679 -1.57079632679 0" xyz="0 0 0"/> <!-- rpy="1.57079632679 0 0" -->
+      <origin rpy="1.57079632679 -1.57079632679 0" xyz="0 0 0"/>
       <parent link="panda_link5"/>
       <child link="panda_link6"/>
@@ -277,5 +213,4 @@
       <dynamics damping="5.0" friction="1.0"/>
     </joint>
-    <!-- panda_link7 -->
     <link name="panda_link7">
       <inertial>
@@ -300,7 +235,6 @@
       </collision>
     </link>
-    <!-- panda_joint7 -->
     <joint name="panda_joint7" type="revolute">
-      <origin rpy="1.57079632679 -0.7854 0" xyz="0.088 0 0"/> <!-- rpy="1.57079632679 0 0" -->
+      <origin rpy="1.57079632679 -0.7854 0" xyz="0.088 0 0"/>
       <parent link="panda_link6"/>
       <child link="panda_link7"/>
@@ -309,7 +243,5 @@
       <dynamics damping="1.0" friction="1.0"/>
     </joint>
-    <!-- panda_link8 -->
     <link name="panda_link8"/>
-    <!-- panda_joint8 -->
     <joint name="panda_joint8" type="fixed">
       <origin rpy="0 0 0" xyz="0 0 0.107"/>
@@ -318,5 +250,4 @@
       <axis xyz="0 0 0"/>
     </joint>
-    <!-- panda_hand -->
     <joint name="panda_hand_joint" type="fixed">
       <parent link="panda_link8"/>
@@ -346,5 +277,4 @@
       </collision>
     </link>
-    <!-- panda_leftfinger -->
     <link name="panda_leftfinger">
       <inertial>
@@ -369,5 +299,4 @@
       </collision>
     </link>
-    <!-- panda_rightfinger -->
     <link name="panda_rightfinger">
       <inertial>
@@ -408,8 +337,6 @@
       <dynamics damping="1.0" friction="1.0"/>
     </joint>
-    <!-- End-Effector frame -->
     <link name="end_effector_frame">
       <inertial>
-        <!-- Dummy inertial parameters to avoid link lumping-->
         <mass value="0.01"/>
         <inertia ixx="0.0001" ixy="0.0" ixz="0.0" iyy="0.0001" iyz="0.0" izz="0.0001"/>

File: franka_env/urdf/panda_ros2control.xacro (robot description, xacro)
@@ -1,55 +1,6 @@
 <?xml version="1.0"?>
-<!--
-# ===================================== COPYRIGHT ===================================== #
-#                                                                                       #
-#  IFRA (Intelligent Flexible Robotics and Assembly) Group, CRANFIELD UNIVERSITY        #
-#  Created on behalf of the IFRA Group at Cranfield University, United Kingdom          #
-#  E-mail: IFRA@cranfield.ac.uk                                                         #
-#                                                                                       #
-#  Licensed under the Apache-2.0 License.                                               #
-#  You may not use this file except in compliance with the License.                     #
-#  You may obtain a copy of the License at: http://www.apache.org/licenses/LICENSE-2.0  #
-#                                                                                       #
-#  Unless required by applicable law or agreed to in writing, software distributed      #
-#  under the License is distributed on an "as-is" basis, without warranties or          #
-#  conditions of any kind, either express or implied. See the License for the specific  #
-#  language governing permissions and limitations under the License.                    #
-#                                                                                       #
-#  IFRA Group - Cranfield University                                                    #
-#  AUTHORS: Mikel Bueno Viso - Mikel.Bueno-Viso@cranfield.ac.uk                         #
-#           Seemal Asif      - s.asif@cranfield.ac.uk                                   #
-#           Phil Webb        - p.f.webb@cranfield.ac.uk                                 #
-#                                                                                       #
-#  Date: July, 2022.                                                                    #
-#                                                                                       #
-# ===================================== COPYRIGHT ===================================== #
-# ===================================== COPYRIGHT ===================================== #
-#                                                                                       #
-#  Some of the information used to build the ROS2 Panda-Robot .urdf files in this ROS2  #
-#  repository has been taken from the following resources:                              #
-#     - frankaemika/franka_ros2 -> https://github.com/frankaemika/franka_ros2.          #
-#       The original files can be found in the franka_description ROS2 package inside   #
-#       he franka_ros2 GitHub repository.                                               #
-#                                                                                       #
-#  AUTHOR: Franka Emika GmbH - support@franka.de                                        #
-#                                                                                       #
-#  Copyright 2021 Franka Emika GmbH                                                     #
-#  (ORIGINAL LICENSE) -> Licensed under the Apache-2.0 License.                         #
-#                                                                                       #
-#  CHANGES MADE:                                                                        #
-#  Robot information/specifications have been taken, and the code has been modified and #
-#  re-organised in accordance with the ros2_RobotSimulation standards.                  #
-#                                                                                       #
-# ===================================== COPYRIGHT ===================================== #
-# ======= CITE OUR WORK ======= #
-# You can cite our work with the following statement:
-# IFRA (2022) ROS2.0 ROBOT SIMULATION. URL: https://github.com/IFRA-Cranfield/ros2_RobotSimulation.
--->
 <robot xmlns:xacro="http://www.ros.org/wiki/xacro">
   <xacro:macro name="panda_ros2control" params="prefix EE_no" >
-    <!-- ROS2_CONTROL tag name: -->
     <xacro:property name="name" value="GazeboSystem"/>
-    <!-- ===== Gazebo ROS2_CONTROL plugin ===== -->
-    <!-- No End-Effector: -->
     <xacro:if value="${EE_no}">
       <gazebo>
@@ -60,12 +11,9 @@
       </gazebo>
     </xacro:if>
-    <!-- ========== ROS2 CONTROL ========== -->
     <ros2_control name="${name}" type="system">
       <hardware>
         <plugin>gazebo_ros2_control/GazeboSystem</plugin>
       </hardware>
-      <!-- panda_joint1 -->
       <joint name="panda_joint1">
-        <!-- <param name="initial_position">0.0</param> -->
         <command_interface name="position">
           <param name="min">-2.8973</param>
@@ -80,7 +28,5 @@
         <state_interface name="effort"/>
       </joint>
-      <!-- panda_joint2 -->
       <joint name="panda_joint2">
-        <!-- <param name="initial_position">-0.785</param> -->
         <command_interface name="position">
           <param name="min">-1.7628</param>
@@ -95,7 +41,5 @@
         <state_interface name="effort"/>
       </joint>
-      <!-- panda_joint3 -->
       <joint name="panda_joint3">
-        <!-- <param name="initial_position">0.0</param> -->
         <command_interface name="position">
           <param name="min">-2.8973</param>
@@ -110,7 +54,5 @@
         <state_interface name="effort"/>
       </joint>
-      <!-- panda_joint4 -->
       <joint name="panda_joint4">
-        <!-- <param name="initial_position">-2.356</param> -->
         <command_interface name="position">
           <param name="min">-3.0718</param>
@@ -125,7 +67,5 @@
         <state_interface name="effort"/>
       </joint>
-      <!-- panda_joint5 -->
       <joint name="panda_joint5">
-        <!-- <param name="initial_position">0.0</param> -->
         <command_interface name="position">
           <param name="min">-2.8973</param>
@@ -140,10 +80,8 @@
         <state_interface name="effort"/>
       </joint>
-      <!-- panda_joint6 -->
       <joint name="panda_joint6">
-        <!-- <param name="initial_position">1.5708</param> -->
         <command_interface name="position">
-          <param name="min">-0.0175</param> <!-- ** -1.5883 -->
-          <param name="max">3.7525</param> <!-- ** 2.1817 -->
+          <param name="min">-0.0175</param>
+          <param name="max">3.7525</param>
         </command_interface>
         <command_interface name="velocity">
@@ -155,10 +93,8 @@
         <state_interface name="effort"/>
       </joint>
-      <!-- panda_joint7 -->
       <joint name="panda_joint7">
-        <!-- <param name="initial_position">0.785</param> -->
         <command_interface name="position">
-          <param name="min">-3.15</param> <!-- ** -3.935 -->
-          <param name="max">3.15</param> <!-- ** 2.365 -->
+          <param name="min">-3.15</param>
+          <param name="max">3.15</param>
         </command_interface>
         <command_interface name="velocity">
@@ -170,5 +106,4 @@
         <state_interface name="effort"/>
       </joint>
-      <!-- panda_finger_joint1 -->
       <joint name="panda_finger_joint1">
         <command_interface name="position">
@@ -184,5 +119,4 @@
         <state_interface name="effort"/>
       </joint>
-      <!-- panda_finger_joint2 -->
       <joint name="panda_finger_joint2">
         <command_interface name="position">
@@ -237,5 +171,4 @@
     <gazebo reference="end_effector_frame_fixed_joint">
       <preserveFixedJoint>true</preserveFixedJoint>
-      <!-- For compatibility with SDFormat < 4.4 -->
       <disableFixedJointLumping>true</disableFixedJointLumping>
     </gazebo>
