Commit message: removed /controller_manager error
New version of ros2_control cannot handle comments inside of URDFs. Removed comments using <!--.*?-->|#.*?$ regex pattern

File: franka_env/urdf/panda_transmission.xacro (robot description, xacro)
@@ -1,49 +1,3 @@
 <?xml version="1.0"?>
-<!--
-# ===================================== COPYRIGHT ===================================== #
-#                                                                                       #
-#  IFRA (Intelligent Flexible Robotics and Assembly) Group, CRANFIELD UNIVERSITY        #
-#  Created on behalf of the IFRA Group at Cranfield University, United Kingdom          #
-#  E-mail: IFRA@cranfield.ac.uk                                                         #
-#                                                                                       #
-#  Licensed under the Apache-2.0 License.                                               #
-#  You may not use this file except in compliance with the License.                     #
-#  You may obtain a copy of the License at: http://www.apache.org/licenses/LICENSE-2.0  #
-#                                                                                       #
-#  Unless required by applicable law or agreed to in writing, software distributed      #
-#  under the License is distributed on an "as-is" basis, without warranties or          #
-#  conditions of any kind, either express or implied. See the License for the specific  #
-#  language governing permissions and limitations under the License.                    #
-#                                                                                       #
-#  IFRA Group - Cranfield University                                                    #
-#  AUTHORS: Mikel Bueno Viso - Mikel.Bueno-Viso@cranfield.ac.uk                         #
-#           Seemal Asif      - s.asif@cranfield.ac.uk                                   #
-#           Phil Webb        - p.f.webb@cranfield.ac.uk                                 #
-#                                                                                       #
-#  Date: July, 2022.                                                                    #
-#                                                                                       #
-# ===================================== COPYRIGHT ===================================== #
-# ===================================== COPYRIGHT ===================================== #
-#                                                                                       #
-#  Some of the information used to build the ROS2 Panda-Robot .urdf files in this ROS2  #
-#  repository has been taken from the following resources:                              #
-#     - frankaemika/franka_ros2 -> https://github.com/frankaemika/franka_ros2.          #
-#       The original files can be found in the franka_description ROS2 package inside   #
-#       he franka_ros2 GitHub repository.                                               #
-#                                                                                       #
-#  AUTHOR: Franka Emika GmbH - support@franka.de                                        #
-#                                                                                       #
-#  Copyright 2021 Franka Emika GmbH                                                     #
-#  (ORIGINAL LICENSE) -> Licensed under the Apache-2.0 License.                         #
-#                                                                                       #
-#  CHANGES MADE:                                                                        #
-#  Robot information/specifications have been taken, and the code has been modified and #
-#  re-organised in accordance with the ros2_RobotSimulation standards.                  #
-#                                                                                       #
-# ===================================== COPYRIGHT ===================================== #
-# ======= CITE OUR WORK ======= #
-# You can cite our work with the following statement:
-# IFRA (2022) ROS2.0 ROBOT SIMULATION. URL: https://github.com/IFRA-Cranfield/ros2_RobotSimulation.
--->
 <robot xmlns:xacro="http://wiki.ros.org/xacro">
   <xacro:macro name="panda_transmission" params="prefix">
